Commit message: Created new ik_fast plugin.

File: src/shi2d2_model/urdf/shi2d2_model.urdf.xacro (robot description, xacro)
@@ -11,5 +11,5 @@
   <xacro:include filename="$(find shi2d2_model)/urdf/gazebo/shi2d2_gazebo_colors.xacro" />
   <xacro:property name="effort" value="1000.0" />
-  <xacro:property name="velocity" value="30.0" />
+  <xacro:property name="velocity" value="100.0" />
   <link name="body_link">
     <inertial>
