Commit message: Cleanup, cleanup, everybody cleanup.

File: src/shi2d2_model/urdf/gazebo/shi2d2_gazebo_plugins.xacro (robot description, xacro)
@@ -3,48 +3,4 @@
     <gazebo>
         <self_collide>1</self_collide>
-        <!-- <plugin filename="gz-sim-joint-state-publisher-system" name="gz::sim::systems::JointStatePublisher">
-        </plugin> -->
-        <!-- <plugin
-            filename="gz-sim-pose-publisher-system"
-            name="gz::sim::systems::PosePublisher">
-            <publish_link_pose>true</publish_link_pose>
-            <use_pose_vector_msg>true</use_pose_vector_msg>
-            <static_publisher>true</static_publisher>
-            <static_update_frequency>1</static_update_frequency>
-        </plugin> -->
-        <!-- <plugin filename="libignition-gazebo-pose-publisher-system"
-            name="ignition::gazebo::systems::PosePublisher">
-            <publish_link_pose>true</publish_link_pose>
-            <publish_sensor_pose>false</publish_sensor_pose>
-            <publish_collision_pose>false</publish_collision_pose>
-            <publish_visual_pose>false</publish_visual_pose>
-            <publish_nested_model_pose>true</publish_nested_model_pose>
-            <use_pose_vector_msg>true</use_pose_vector_msg>
-            <update_frequency>0</update_frequency>
-            <static_publisher>true</static_publisher>
-            <static_update_frequency>60</static_update_frequency>
-        </plugin>  -->
-        <!-- <plugin filename="libignition-gazebo-pose-publisher-system" name="ignition::gazebo::systems::PosePublisher">
-            <publish_link_pose>false</publish_link_pose>
-            <publish_model_pose>false</publish_model_pose>
-            <publish_nested_model_pose>true</publish_nested_model_pose>
-            <use_pose_vector_msg>true</use_pose_vector_msg>
-        </plugin> -->
-        <!-- <plugin filename="ignition-gazebo-joint-state-publisher-system" name="ignition::gazebo::systems::JointStatePublisher">
-            <topic>joint_states</topic>
-            <joint_name>head_upper_neck_joint</joint_name>
-            <joint_name>upper_neck_lower_neck_joint</joint_name>
-            <joint_name>lower_neck_body_joint</joint_name>
-            <joint_name>left_upper_hip_body_joint</joint_name>
-            <joint_name>left_lower_hip_left_upper_hip_joint</joint_name>
-            <joint_name>left_upper_leg_left_lower_hip_joint</joint_name>
-            <joint_name>left_lower_leg_left_upper_leg_joint</joint_name>
-            <joint_name>left_foot_left_lower_leg_joint</joint_name>
-            <joint_name>right_upper_hip_body_joint</joint_name>
-            <joint_name>right_lower_hip_right_upper_hip_joint</joint_name>
-            <joint_name>right_upper_leg_right_lower_hip_joint</joint_name>
-            <joint_name>right_lower_leg_right_upper_leg_joint</joint_name>
-            <joint_name>right_foot_right_lower_leg_joint</joint_name>
-        </plugin> -->
         <plugin filename="ignition-gazebo-pose-publisher-system" name="ignition::gazebo::systems::PosePublisher">
             <publish_link_pose>false</publish_link_pose>
@@ -52,6 +8,4 @@
             <publish_nested_model_pose>false</publish_nested_model_pose>
             <use_pose_vector_msg>true</use_pose_vector_msg>
-            <!-- <static_publisher>true</static_publisher> -->
-            <!-- <static_update_frequency>1</static_update_frequency> -->
         </plugin>
         <plugin filename="ignition-gazebo-odometry-publisher-system" name="ignition::gazebo::systems::OdometryPublisher">
@@ -64,10 +18,4 @@
             <robot_param_node>robot_state_publisher</robot_param_node>
         </plugin>
-            <!-- <controller_manager_name>controller_manager</controller_manager_name>   -->
-        <!-- <plugin
-            filename="ignition-gazebo-joint-position-controller-system"
-            name="ignition::gazebo::systems::JointPositionController">
-            <joint_name>head_upper_neck_joint</joint_name>
-        </plugin>     -->
     </gazebo>
 </robot>

File: src/shi2d2_model/urdf/shi2d2_model.urdf.xacro (robot description, xacro)
@@ -9,16 +9,4 @@
   <xacro:property name="effort" value="1000.0" />
   <xacro:property name="velocity" value="30.0" />
-  <!-- <link name="world"/>
-  <joint name="body_world_joint" type="floating">
-    <origin rpy="0 0 0" xyz="0 0 1"/>
-    <parent link="world"/>
-    <child link="body_link"/>
-  </joint> -->
-  <!-- <link name="shi2d2"></link>
-  <joint name="virtual_joint" type="fixed">
-      <parent link="shi2d2" />
-      <child link="body_link" />
-      <origin rpy="0 0 0" xyz="0 0 0" />
-  </joint> -->
   <link name="body_link">
     <inertial>

Commit message: Added telemetry and sensors to get robot state and center of mass estimate.

File: src/shi2d2_model/urdf/gazebo/shi2d2_gazebo_plugins.xacro (robot description, xacro)
@@ -8,13 +8,17 @@
       <robot_param_node>robot_state_publisher</robot_param_node>
     </plugin>
-    <plugin filename="gz-sim-pose-publisher-system" name="gz::sim::systems::PosePublisher">
+    <!-- <plugin filename="gz-sim-pose-publisher-system" name="gz::sim::systems::PosePublisher">
       <publish_link_pose>false</publish_link_pose>
       <publish_model_pose>true</publish_model_pose>
       <publish_nested_model_pose>false</publish_nested_model_pose>
       <use_pose_vector_msg>true</use_pose_vector_msg>
-    </plugin>
+    </plugin> -->
     <plugin filename="gz-sim-odometry-publisher-system" name="gz::sim::systems::OdometryPublisher">
       <odom_frame>world</odom_frame>
-      <robot_base_frame>body_link</robot_base_frame>
+      <!-- <robot_base_frame>body_link</robot_base_frame> -->
+      <robot_base_frame>com_link</robot_base_frame>
+      <dimensions>3</dimensions>
+      <xyz_offset>0 0 0</xyz_offset>
+      <rpy_offset>0 0 0</rpy_offset>
     </plugin>
     <plugin filename="gz-sim-sensors-system" name="gz::sim::systems::Sensors">

File: src/shi2d2_model/urdf/gazebo/shi2d2_gazebo_sensors.xacro (robot description, xacro)
@@ -1,5 +1,5 @@
 <?xml version="1.0" ?>
 <robot xmlns:xacro="http://wiki.ros.org/xacro">
-  <gazebo reference="body_link">
+  <gazebo reference="com_link">
     <sensor name="imu_sensor" type="imu">
       <always_on>true</always_on>

File: src/shi2d2_model/urdf/shi2d2_model.urdf.xacro (robot description, xacro)
@@ -11,4 +11,31 @@
   <xacro:property name="effort" value="1000.0" />
   <xacro:property name="velocity" value="100.0" />
+  <!-- virtual center of mass link and joint -->
+  <link name="com_link">
+    <inertial>
+        <origin xyz="0 0 0" rpy="0 0 0" />
+        <mass value="0.0001" />
+        <inertia ixx="0.0001" ixy="0" ixz="0" iyy="0.0001" iyz="0" izz="0.0001" />
+    </inertial>
+    <visual>
+        <origin xyz="0 0 0" rpy="0 0 0" />
+        <geometry>
+          <sphere radius="0.01" />
+        </geometry>
+        <material name="red">
+          <color rgba="1 0 0 1" />
+        </material>
+    </visual>
+    <collision>
+        <origin xyz="0 0 0" rpy="0 0 0" />
+    </collision>
+  </link>
+  <joint name="com_body_joint" type="fixed">
+    <!-- specifies location of center of mass relative to body link origin -->
+    <!-- curently derived from the negative of the xyz attribute of body_link's inertial property -->
+    <origin xyz="0.13606 0 -0.011359" rpy="0 0 0" />
+    <parent link="com_link" />
+    <child link="body_link" />
+  </joint>
   <link name="body_link">
     <inertial>
